File: hw/project/_autosave-peripherals.kicad_sch (KiCad schematic)
At the start: 32 parts, among them J1 XT60PW-M, J2 Hall, J3 SWD, J4 Serial, J5 7461001, J6 7461001, J7 7461001

Commit message: Distinguish between hierarchical VM_IN and global VM
Changed lines of the file:
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@@
 		)
 	)
-	(text_box "Serial \n\nUses PA9 (USART1_TX) & PA10 (USART1_RX)"
+	(text_box "Serial \n\nUses PA9 & PA10, label pins with TX & RX"
 		(exclude_from_sim no)
 		(at 119.38 26.67 0)
