File: hw/project/peripherals.kicad_sch (KiCad schematic)
At the start: 70 parts, among them J1 XT60PW-M, J2 Hall, J3 SWD, J4 Serial, J5 7461001, J6 7461001, J7 7461001, J9 CONN HEADER VERT 4POS 2.5MM, SW3 RESET, SW4 RESET, U2 ATA6561-GAQW-N

Commit message: Reorg LEDs
Parts:
- removed C54: 1nF, Capacitor_SMD:C_0603_1608Metric, symbol Device:C_Small
- removed D22, D25, D26: 2Vf, LED_SMD:LED_0603_1608Metric_Pad1.05x0.95mm_HandSolder, symbol Device:LED
- removed R74: 100k, symbol Device:R_Small_US
- removed R75: 120, symbol Device:R_Small_US
- removed R76: 200, symbol Device:R_Small_US
- removed R79, R83: 130, symbol Device:R_Small_US
- removed SW4: RESET, SWT0220_016016GSA:SW_SWT0220-016016GSA_REVA, symbol Switch:SW_Push
- SW3: value RESET -> USER
Connections:
- net FAULT renamed FAULT_LED
- net LED1 renamed SYS_LED1
- net LED2 renamed SYS_LED2
- net USER/WAKE renamed USER_SW
Other:
- note added: "Power Status LEDs"
- note added: "System LEDs"
- note added: "change to blue"
- note added: "change to white"
- note added: "change to yellow"
- note removed: "Extra leds can be used for rx/tx or whatever"
- note removed: "evspin had two of these, one for wake and another for idk what"
- moved on the sheet: C53, D19, D20, D21, D23, D24, D27, D28, R71, R72, R73, R77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
