File: hw/project/drive.kicad_sch (KiCad schematic)
At the start: 63 parts, among them Q3 STL110N10F7, Q4 STL110N10F7, Q5 STL110N10F7, Q6 STL110N10F7, Q7 STL110N10F7, Q8 STL110N10F7

Commit message: Finalize drive sheet
Parts:
- removed C32: 1uF/25V, symbol Device:C_Small
- removed C34: 220nF/100V, symbol Device:C_Small
- removed D3, D4: BAT48RL, Diode_THT:D_DO-35_SOD27_P7.62mm_Horizontal, symbol Diode:BAT48RL
- removed Q3, Q4: STL110N10F7, symbol Transistor_FET:Q_NMOS_DGS
- removed R20, R27: 2m/2W, symbol Device:R_Shunt_US
- removed R22, R23: 33, symbol Device:R_Small_US
- removed R24, R25, R26: 0, symbol Device:R_Small_US
- removed R30, R31: 33, Resistor_SMD:R_0603_1608Metric, symbol Device:R_Small_US
- added C39: 1uF/25V, Capacitor_SMD:C_0603_1608Metric, symbol Device:C_Small
- added C42: 220nF/100V, Capacitor_SMD:C_0603_1608Metric, symbol Device:C_Small
- added D17, D19: BAT48JFILM, Diode_SMD:D_SOD-323, symbol Diode:BAT48RL
- added Q10, Q9: STL110N10F7, STL110N10F7:MOSFET_10N10F7_STM, symbol Transistor_FET:Q_NMOS_DGS
- added R85, R86: 2m/3W, Resistor_SMD:R_2512_6332Metric, symbol Device:R_Shunt_US
- added R87, R88, R89, R90, R91, R92: 10, Resistor_SMD:R_0603_1608Metric, symbol Device:R_Small_US
- added R93: 0, Resistor_SMD:R_0603_1608Metric, symbol Device:R_Small_US
- C40: value 220nF -> 220nF/100V
- D16, D5, D6, D7: value BAT48RL -> BAT48JFILM; footprint Diode_THT:D_DO-35_SOD27_P7.62mm_Horizontal -> Diode_SMD:D_SOD-323
- D35, D36, D37, D38, D39, D40: value BAT30K -> BAT30KFILM
- R38, R39: value 33 -> 0
Connections:
- net BOOT1: now also C39.2
- net GHS1: now also D17.1 (K), R90.1; no longer D16.1 (K)
- net GHS2: now also R91.1
- net GHS3: now also D7.1 (K), R92.1; no longer D6.1 (K), R38.1
- net GLS1: now also D19.1 (K), R87.1
- net GLS2: now also D6.1 (K), R88.1
- net GLS3: now also D16.1 (K), R89.1; no longer D7.1 (K), R39.1
- net GND: no longer C37.1, C40.1, R28.4, R35.4, R36.4, R43.4
- net OUT1: now also C39.1, R93.1
- net U: now also Q10.1 (D), Q9.3 (S), R93.2
- net VM: now also C42.2, Q9.1 (D)
- net VSHUNT_U+: now also R85.2, R86.2
- net VSHUNT_U-: now also R85.3, R86.3
- net at Q8.2 (G), R41.2: now also R89.2; no longer R39.2
- net at Q5.2 (G), R32.2: now also R91.2
- net at Q7.2 (G), R40.2: now also R92.2; no longer R38.2
- net at D6.2 (A): now also R33.1; no longer R40.1
- net at Q6.2 (G), R33.2: now also R88.2
- net at D7.2 (A): now also R40.1; no longer R41.1
- net at D16.2 (A): now also R41.1
- new net: Q9.2 (G), R39.2, R90.2
- new net: Q10.3 (S), R85.1, R86.1
- new net: D19.2 (A), R38.1
- new net: D17.2 (A), R39.1
- new net: Q10.2 (G), R38.2, R87.2
- new net PGND: C37.1, C40.1, C42.1, R28.4, R35.4, R36.4, R43.4, R85.4, R86.4
Other:
- note removed: "C0G/NP0 required!! so cant reuse hall sensor's 1nF, but can just it for all"
- note removed: "PGND?"
- moved on the sheet: C33, C36, D37, D38, D39, D40, R28, R35, R36, R43, R70, R74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

Commit message: Prep to revamp power sheet
Changed lines of the file:
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@@
 		)
 	)
-	(text_box "Transfer Function: V_OUT = V_DAC - ( |G_inverting| * V_SHUNT )\n\n- To keep 0A midpoint at VDD / 2 = 1.65V, config DAC at 2048\n- G=-63 for bench testing (2A) & G=-31 for reg. riding (<50A)"
+	(text_box "Transfer Function: V_OUT = V_DAC - ( |G_inverting| * V_SHUNT )\n- To keep 0A midpoint at VDD / 2 = 1.65V, config DAC at 2048\n- G=-63 (bench testing): {-26, 26} [A] -> {0.012, 3.288} [V]\n- G=-31 (regular riding): {-53, 53} [A] -> {0.007, 3.293} [V]"
 		(exclude_from_sim no)
 		(at 246.38 109.2201 0)
